Commit message: some updates

File: examples/floatingBase/rsc/1dof_float2.urdf (robot description, URDF)
Before this commit: robot 1dof, 3 links, 2 joints
Links:
- added link link3, mass 1; collision cylinder length=0.250 radius=0.01; visual cylinder length=0.250 radius=0.01
Joints:
- added joint Joint3: type revolute, parent trunk, child link3, origin xyz=0 -0.06 0.0 rpy=0 0 0, axis 0 -1 0
- joint Joint2: axis 0 1 0 -> 1 0 0

Commit message: inverse dynamics is working

File: examples/floatingBase/rsc/1dof_float2.urdf (robot description, URDF)
Before this commit: robot 1dof, 4 links, 3 joints
Joints:
- joint Joint3: axis 0 -1 0 -> 0 1 0; origin xyz=0 -0.06 0.0 rpy=0 0 0 -> xyz=0 -0.06 0.0 rpy=0 0 3.14159265359

Commit message: small changes

File: examples/floatingBase/rsc/1dof_float2.urdf (robot description, URDF)
Before this commit: robot 1dof, 4 links, 3 joints
Links:
- added link link4, mass 1; collision cylinder length=0.250 radius=0.01; visual cylinder length=0.250 radius=0.01
- link link3: geometry collision sphere radius=0.01; visual sphere radius=0.01
Joints:
- added joint Joint4: type revolute, parent trunk, child link4, origin xyz=0 -0.06 0.0 rpy=0 0 3.14159265359, axis 0 1 0
- joint Joint3: axis 0 1 0 -> (none); origin xyz=0 -0.06 0.0 rpy=0 0 3.14159265359 -> xyz=0 0 0.250 rpy=0 0 0; parent trunk -> link2; type revolute -> fixed
