Commit message: some small changes

File: examples/fixedBase/rsc/1dof2.urdf (robot description, URDF)
Before this commit: robot 1dof, 6 links, 5 joints
Links:
- added link link5, mass 1; collision cylinder length=0.250 radius=0.01; visual cylinder length=0.250 radius=0.01
- added link link6, mass 1; collision sphere radius=0.01; visual sphere radius=0.01
- link link3: geometry collision sphere radius=0.01; visual sphere radius=0.01
Joints:
- added joint Joint5: type revolute, parent link4, child link5, origin xyz=0 0 0.250 rpy=0 0 3.14159265359, axis 1 0 0
- added joint Joint6: type fixed, parent link5, child link6, origin xyz=0 0 0.250 rpy=0 0 0
- joint Joint3: axis 0 -1 0 -> (none); origin xyz=0 -0.06 0 rpy=0 0 0 -> xyz=0 0 0.250 rpy=0 0 0; parent trunk -> link2; type revolute -> fixed
- joint Joint4: axis 1 0 0 -> 0 1 0; origin xyz=0 0 0.250 rpy=0 0 0 -> xyz=0 -0.06 0 rpy=0 0 3.14159265359; parent link3 -> trunk

Commit message: inverse and forward kinematics added

File: examples/fixedBase/rsc/1dof2.urdf (robot description, URDF)
Before this commit: robot 1dof, 8 links, 7 joints
Joints:
- joint Joint4: origin xyz=0 -0.06 0 rpy=0 0 3.14159265359 -> xyz=0 -0.06 0 rpy=0 0 0
- joint Joint5: origin xyz=0 0 0.250 rpy=0 0 3.14159265359 -> xyz=0 0 0.250 rpy=0 0 0

File: examples/floatingBase/rsc/1dof_float2.urdf (robot description, URDF)
Before this commit: robot 1dof, 5 links, 4 joints
Links:
- added link link5, mass 1; collision cylinder length=0.250 radius=0.01; visual cylinder length=0.250 radius=0.01
- added link link6, mass 1; collision sphere radius=0.01; visual sphere radius=0.01
Joints:
- added joint Joint5: type revolute, parent link4, child link5, origin xyz=0 0 0.250 rpy=0 0 0, axis 0 -1 0
- added joint Joint6: type fixed, parent link5, child link6, origin xyz=0 0 0.250 rpy=0 0 0
- joint Joint4: axis 0 1 0 -> -1 0 0; origin xyz=0 -0.06 0.0 rpy=0 0 3.14159265359 -> xyz=0 -0.06 0.0 rpy=0 0 0

File: examples/kinematicTests/rsc/1dof.urdf (robot description, URDF)
Before this commit: robot 1dof, 4 links, 3 joints
Links:
- added link link3, mass 1; collision sphere radius=0.01; visual sphere radius=0.01
Joints:
- added joint Joint3: type fixed, parent link2, child link3, origin xyz=0 0 0.250 rpy=0 0 0

File: examples/kinematicTests/rsc/1dof2.urdf (robot description, URDF)
Before this commit: robot 1dof, 6 links, 5 joints
Links:
- added link link5, mass 1; collision cylinder length=0.250 radius=0.01; visual cylinder length=0.250 radius=0.01
- added link link6, mass 1; collision sphere radius=0.01; visual sphere radius=0.01
- link link3: geometry collision sphere radius=0.01; visual sphere radius=0.01
Joints:
- added joint Joint5: type revolute, parent link4, child link5, origin xyz=0 0 0.250 rpy=0 0 0, axis 1 0 0
- added joint Joint6: type fixed, parent link5, child link6, origin xyz=0 0 0.250 rpy=0 0 0
- joint Joint3: axis 0 -1 0 -> (none); origin xyz=0 -0.06 0 rpy=0 0 0 -> xyz=0 0 0.250 rpy=0 0 0; parent trunk -> link2; type revolute -> fixed
- joint Joint4: axis 1 0 0 -> 0 1 0; origin xyz=0 0 0.250 rpy=0 0 0 -> xyz=0 -0.06 0 rpy=0 0 0; parent link3 -> trunk
