Commit message: Axis sign added in kinematics

File: examples/quadruped/rsc/urdf/quadruped2.urdf (robot description, URDF)
Before this commit: robot tekirV3, 17 links, 16 joints
Joints:
- joint footFrame_lb: origin xyz=0 0 -0.224282 rpy=0 0.52359877559 0 -> xyz=-0.053565 0 -0.317060 rpy=0 0.52359877559 0
- joint footFrame_lf: origin xyz=0 0 -0.224282 rpy=0 0.52359877559 0 -> xyz=-0.053565 0 -0.317060 rpy=0 0.52359877559 0
- joint footFrame_rb: origin xyz=0 0 -0.224282 rpy=0 0.52359877559 0 -> xyz=-0.053565 0 -0.317060 rpy=0 0.52359877559 0
- joint footFrame_rf: origin xyz=0 0 -0.224282 rpy=0 0.52359877559 0 -> xyz=-0.053565 0 -0.317060 rpy=0 0.52359877559 0
