Commit message: GO2 urdfs updated

File: examples/rsc/go2/urdf/go2_1.urdf (robot description, URDF)
Before this commit: robot go2, 18 links, 17 joints
Links:
- removed link imu_link
Joints:
- removed joint imu_joint
- joint FL_foot_joint: origin xyz=0 0 -0.213 rpy=0 0.5617198 0 -> xyz=-0.011 0 -0.232052 rpy=0 0.5617198 0
- joint FR_foot_joint: origin xyz=0 0 -0.213 rpy=0 0.5617198 0 -> xyz=-0.011 0 -0.232052 rpy=0 0.5617198 0
- joint RL_foot_joint: origin xyz=0 0 -0.213 rpy=0 0.5617198 0 -> xyz=-0.011 0 -0.232052 rpy=0 0.5617198 0
- joint RR_foot_joint: origin xyz=0 0 -0.213 rpy=0 0.5617198 0 -> xyz=-0.011 0 -0.232052 rpy=0 0.5617198 0
